File: Themis.sch (KiCad schematic (older format))
At the start: 35 parts, among them J10 Conn_01x01, J11 Conn_01x01, J12 Conn_01x01, J13 Conn_01x01, J17 SMA, J18 Conn_01x01, J20 Conn_01x01, J5 Conn_01x05, J7 SMA, J8 SMA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

Commit message: upgrade to Kicad 5.x
Parts:
- C1, C2, C3, C4, C5: symbol C_Small -> Themis-rescue:C_Small
- D1, D2, D3, D4: symbol D_Small_ALT -> Themis-rescue:D_Small_ALT
- J10, J11, J12, J13, J18, J20: symbol Conn_01x01 -> Themis-rescue:Conn_01x01
- J17, J7, J8: symbol Conn_Coaxial -> Themis-rescue:Conn_Coaxial
- J5: symbol Conn_01x05 -> Themis-rescue:Conn_01x05
- R1, R10, R11, R12, R13, R2, R3, R4, R5, R6, R7, R8, R9: symbol R_Small -> Themis-rescue:R_Small
- T1, T2: symbol Transformer_1P_1S -> Themis-rescue:Transformer_1P_1S
- U1: symbol LMC6482 -> Themis-rescue:LMC6482
